File: EE/tamagotchi/Pressure.kicad_sch (KiCad schematic)
At the start: 4 parts, among them U3 MPL3115A2

Commit message: WIP - Overall Cleanup, Power Change
Added expected loads for power in schematic.
Changed power arch to use existing design that appears to work.
Removed rear backlight LEDs - shouldn't be necessary.
Other:
- note added: "2mA during acq/conv"
- note added: "TODO 10u"
Changed lines of the file:
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@@
 	(generator_version "9.0")
 	(paper "A4")
+	(text "2mA during acq/conv"
+		(exclude_from_sim no)
+		(at 162.052 80.264 0)
+		(effects
+			(font
+				(size 1.27 1.27)
+			)
+		)
+	)
+	(text "TODO 10u"
+		(exclude_from_sim no)
+		(at 114.3 86.614 0)
+		(effects
+			(font
+				(size 1.27 1.27)
+			)
+		)
+	)
 	(junction
 		(at 143.51 78.74)
